Commit message: Correct S6LR assembly and add world locomotion

File: public/models/s6lr/hexapod.urdf (robot description, URDF)
Before this commit: robot s6lr_hexapod, 19 links, 18 joints
Links:
- link femur_1: mass 0.15 -> None; geometry visual mesh filename=xml_Files/Servo femur.stl scale=0.001 0.001 0.001; visual mesh filename=xml_Files/Servo tibia.stl scale=0.001 0.001 0.001
- link femur_2: mass 0.15 -> None; geometry visual mesh filename=xml_Files/Servo femur.stl scale=0.001 -0.001 0.001; visual mesh filename=xml_Files/Servo tibia.stl scale=0.001 -0.001 0.001
- link femur_3: mass 0.15 -> None; geometry visual mesh filename=xml_Files/Servo femur.stl scale=0.001 0.001 0.001; visual mesh filename=xml_Files/Servo tibia.stl scale=0.001 0.001 0.001
- link femur_4: mass 0.15 -> None; geometry visual mesh filename=xml_Files/Servo femur.stl scale=0.001 -0.001 0.001; visual mesh filename=xml_Files/Servo tibia.stl scale=0.001 -0.001 0.001
- link femur_5: mass 0.15 -> None; geometry visual mesh filename=xml_Files/Servo femur.stl scale=0.001 0.001 0.001; visual mesh filename=xml_Files/Servo tibia.stl scale=0.001 0.001 0.001
- link femur_6: mass 0.15 -> None; geometry visual mesh filename=xml_Files/Servo femur.stl scale=0.001 -0.001 0.001; visual mesh filename=xml_Files/Servo tibia.stl scale=0.001 -0.001 0.001
- link hip_1: mass 0.05 -> None; geometry visual mesh filename=xml_Files/hip frame right mid.stl scale=0.001 0.001 0.001
- link hip_2: mass 0.05 -> None; geometry visual mesh filename=xml_Files/hip frame right mid.stl scale=0.001 -0.001 0.001
- link hip_3: mass 0.05 -> None; geometry visual mesh filename=xml_Files/hip frame right mid.stl scale=0.001 0.001 0.001
- link hip_4: mass 0.05 -> None; geometry visual mesh filename=xml_Files/hip frame right mid.stl scale=0.001 -0.001 0.001
- link hip_5: mass 0.05 -> None; geometry visual mesh filename=xml_Files/hip frame right mid.stl scale=0.001 0.001 0.001
- link hip_6: mass 0.05 -> None; geometry visual mesh filename=xml_Files/hip frame right mid.stl scale=0.001 -0.001 0.001
- link tibia_1: mass 0.1 -> None; geometry visual mesh filename=xml_Files/tibia base.stl scale=0.001 0.001 0.001; visual mesh filename=xml_Files/tibia frame A.stl scale=0.001 0.001 0.001
- link tibia_2: mass 0.1 -> None; geometry visual mesh filename=xml_Files/tibia base.stl scale=0.001 -0.001 0.001; visual mesh filename=xml_Files/tibia frame A.stl scale=0.001 -0.001 0.001
- link tibia_3: mass 0.1 -> None; geometry visual mesh filename=xml_Files/tibia base.stl scale=0.001 0.001 0.001; visual mesh filename=xml_Files/tibia frame A.stl scale=0.001 0.001 0.001
- link tibia_4: mass 0.1 -> None; geometry visual mesh filename=xml_Files/tibia base.stl scale=0.001 -0.001 0.001; visual mesh filename=xml_Files/tibia frame A.stl scale=0.001 -0.001 0.001
- link tibia_5: mass 0.1 -> None; geometry visual mesh filename=xml_Files/tibia base.stl scale=0.001 0.001 0.001; visual mesh filename=xml_Files/tibia frame A.stl scale=0.001 0.001 0.001
- link tibia_6: mass 0.1 -> None; geometry visual mesh filename=xml_Files/tibia base.stl scale=0.001 -0.001 0.001; visual mesh filename=xml_Files/tibia frame A.stl scale=0.001 -0.001 0.001
- link torso: mass 2.0 -> None; geometry visual mesh filename=xml_Files/base roll.stl scale=0.001 0.001 0.001; visual mesh filename=xml_Files/camera holder A.stl scale=0.001 0.001 0.001
Joints:
- joint femur_joint_1: limit lower=-1.0 upper=1.0 effort=5.0 velocity=3.0 -> lower=-3 upper=3 effort=5 velocity=3; origin xyz=0 0.028 -0.0415 rpy=0 0 0 -> xyz=0 0.024 0.0115 rpy=0 0 0
- joint femur_joint_2: limit lower=-1.0 upper=1.0 effort=5.0 velocity=3.0 -> lower=-3 upper=3 effort=5 velocity=3; origin xyz=0 -0.028 -0.0415 rpy=0 0 0 -> xyz=0 -0.024 0.0115 rpy=0 0 0
- joint femur_joint_3: limit lower=-1.0 upper=1.0 effort=5.0 velocity=3.0 -> lower=-3 upper=3 effort=5 velocity=3; origin xyz=0 0.028 -0.0415 rpy=0 0 0 -> xyz=0 0.024 0.0115 rpy=0 0 0
- joint femur_joint_4: limit lower=-1.0 upper=1.0 effort=5.0 velocity=3.0 -> lower=-3 upper=3 effort=5 velocity=3; origin xyz=0 -0.028 -0.0415 rpy=0 0 0 -> xyz=0 -0.024 0.0115 rpy=0 0 0
- joint femur_joint_5: limit lower=-1.0 upper=1.0 effort=5.0 velocity=3.0 -> lower=-3 upper=3 effort=5 velocity=3; origin xyz=0 0.028 -0.0415 rpy=0 0 0 -> xyz=0 0.024 0.0115 rpy=0 0 0
- joint femur_joint_6: limit lower=-1.0 upper=1.0 effort=5.0 velocity=3.0 -> lower=-3 upper=3 effort=5 velocity=3; origin xyz=0 -0.028 -0.0415 rpy=0 0 0 -> xyz=0 -0.024 0.0115 rpy=0 0 0
- joint hip_joint_1: limit lower=-1.0 upper=1.0 effort=5.0 velocity=3.0 -> lower=-1 upper=1 effort=5 velocity=3; origin xyz=-0.050 -0.0035 0 rpy=0 0 0 -> xyz=-0.05 0.0245 -0.0415 rpy=0 0 0
- joint hip_joint_2: limit lower=-1.0 upper=1.0 effort=5.0 velocity=3.0 -> lower=-1 upper=1 effort=5 velocity=3; origin xyz=-0.050 0.0035 0 rpy=0 0 0 -> xyz=-0.05 -0.0245 -0.0415 rpy=0 0 0
- joint hip_joint_3: limit lower=-1.0 upper=1.0 effort=5.0 velocity=3.0 -> lower=-1 upper=1 effort=5 velocity=3; origin xyz=0 0 0 rpy=0 0 0 -> xyz=0 0.028 -0.0415 rpy=0 0 0
- joint hip_joint_4: limit lower=-1.0 upper=1.0 effort=5.0 velocity=3.0 -> lower=-1 upper=1 effort=5 velocity=3; origin xyz=0 0 0 rpy=0 0 0 -> xyz=0 -0.028 -0.0415 rpy=0 0 0
- joint hip_joint_5: limit lower=-1.0 upper=1.0 effort=5.0 velocity=3.0 -> lower=-1 upper=1 effort=5 velocity=3; origin xyz=0.050 -0.0035 0 rpy=0 0 0 -> xyz=0.05 0.0245 -0.0415 rpy=0 0 0
- joint hip_joint_6: limit lower=-1.0 upper=1.0 effort=5.0 velocity=3.0 -> lower=-1 upper=1 effort=5 velocity=3; origin xyz=0.050 0.0035 0 rpy=0 0 0 -> xyz=0.05 -0.0245 -0.0415 rpy=0 0 0
- joint tibia_joint_1: limit lower=0 upper=1.57 effort=5.0 velocity=3.0 -> lower=-3 upper=3 effort=5 velocity=3; origin xyz=0.0175 0.0405 0.024 rpy=0 0 0 -> xyz=0 0.0165 0.054 rpy=0 0 0
- joint tibia_joint_2: limit lower=-1.0 upper=1.0 effort=5.0 velocity=3.0 -> lower=-3 upper=3 effort=5 velocity=3; origin xyz=0.0175 -0.0405 0.024 rpy=0 0 0 -> xyz=0 -0.0165 0.054 rpy=0 0 0
- joint tibia_joint_3: limit lower=-1.0 upper=1.0 effort=5.0 velocity=3.0 -> lower=-3 upper=3 effort=5 velocity=3; origin xyz=0.0175 0.0405 0.024 rpy=0 0 0 -> xyz=0 0.0165 0.054 rpy=0 0 0
- joint tibia_joint_4: limit lower=-1.0 upper=1.0 effort=5.0 velocity=3.0 -> lower=-3 upper=3 effort=5 velocity=3; origin xyz=0.0175 -0.0405 0.024 rpy=0 0 0 -> xyz=0 -0.0165 0.054 rpy=0 0 0
- joint tibia_joint_5: limit lower=-1.0 upper=1.0 effort=5.0 velocity=3.0 -> lower=-3 upper=3 effort=5 velocity=3; origin xyz=0.0175 0.0405 0.024 rpy=0 0 0 -> xyz=0 0.0165 0.054 rpy=0 0 0
- joint tibia_joint_6: limit lower=-1.0 upper=1.0 effort=5.0 velocity=3.0 -> lower=-3 upper=3 effort=5 velocity=3; origin xyz=0.0175 -0.0405 0.024 rpy=0 0 0 -> xyz=0 -0.0165 0.054 rpy=0 0 0
